Commit message: added inertial properties to URDF for improved simulation accuracy

File: my_robot_description/urdf/common_properties.xacro (robot description, xacro)
@@ -7,3 +7,34 @@
         <color rgba="0.5 0.5 0.5 1" />
     </material>
+    <!-- https://en.wikipedia.org/wiki/List_of_moments_of_inertia#List_of_3D_inertia_tensors -->
+    <xacro:macro name="box_inertia" params="m l w h xyz rpy">
+        <inertial>
+            <origin xyz="${xyz}" rpy="${rpy}" />
+            <mass value="${m}" />
+            <!--for a solid cuboid-->
+            <inertia ixx="${(m/12) * (h*h + l*l)}" ixy="0" ixz="0"
+                     iyy="${(m/12) * (w*w + h*h)}" iyz="0"
+                     izz="${(m/12) * (w*w + l*l)}" />   <!--only need the upper triangle matrix-->
+        </inertial>
+    </xacro:macro>
+    <xacro:macro name="cylinder_inertia" params="m r l xyz rpy">
+        <inertial>
+            <origin xyz="${xyz}" rpy="${rpy}" />
+            <mass value="${m}" />
+            <!--for a solid cylinder-->
+            <inertia ixx="${(m/12) * (3*r*r + l*l)}" ixy="0" ixz="0"
+                     iyy="${(m/12) * (3*r*r + l*l)}" iyz="0"
+                     izz="${(m/2) * (r*r)}" />
+        </inertial>
+    </xacro:macro>
+    <xacro:macro name="sphere_inertia" params="m r xyz rpy">
+        <inertial>
+            <origin xyz="${xyz}" rpy="${rpy}" />
+            <mass value="${m}" />
+            <!--for a solid sphere-->
+            <inertia ixx="${0.4*m * r*r}" ixy="0" ixz="0"
+                     iyy="${0.4*m * r*r}" iyz="0"
+                     izz="${0.4*m * r*r}" />
+        </inertial>
+    </xacro:macro>
 </robot>

File: my_robot_description/urdf/mobile_base.xacro (robot description, xacro)
@@ -12,7 +12,9 @@
                 <box size="${base_length} ${base_width} ${base_height}" />  <!-- lenght width height. in metric system . meters-->
             </geometry>
-            <origin xyz="0 0 0.1" rpy="0 0 0" />    <!--roll pitch yaw . radian-->
+            <origin xyz="0 0 ${base_height / 2.0}" rpy="0 0 0" />    <!--roll pitch yaw . radian-->
             <material name="blue" />                <!--we used the material tag-->
         </visual>
+        <xacro:box_inertia m="5.0" l="${base_length}" w="${base_width}" h="${base_height}"
+                           xyz="${base_height / 2.0}" rpy="0 0 0" />
     </link>
     <!--function. params not mandatory-->
@@ -26,4 +28,6 @@
                 <material name="gray" />
             </visual>
+            <xacro:cylinder_inertia m="1.0" r="${wheel_radius}" l="${wheel_length}"
+                                 xyz="0 0 0" rpy="${pi / 2.0} 0 0" />
         </link>
     </xacro:macro>
@@ -38,4 +42,6 @@
             <material name="gray" />
         </visual>
+        <xacro:sphere_inertia m="0.5" r="${wheel_radius / 2.0}"
+                              xyz="0 0 0" rpy="0 0 0" />
     </link>
     <joint name="base_joint" type="fixed">

Commit message: created new bringup pkg, recreated launch file

File: my_robot_description/urdf/common_properties.xacro (robot description, xacro)
@@ -13,7 +13,7 @@
             <mass value="${m}" />
             <!--for a solid cuboid-->
-            <inertia ixx="${(m/12) * (h*h + l*l)}" ixy="0" ixz="0"
-                     iyy="${(m/12) * (w*w + h*h)}" iyz="0"
-                     izz="${(m/12) * (w*w + l*l)}" />   <!--only need the upper triangle matrix-->
+            <inertia ixx="${(m/12.0) * (h*h + l*l)}" ixy="0" ixz="0"
+                     iyy="${(m/12.0) * (w*w + h*h)}" iyz="0"
+                     izz="${(m/12.0) * (w*w + l*l)}" />   <!--only need the upper triangle matrix-->
         </inertial>
     </xacro:macro>
@@ -23,7 +23,7 @@
             <mass value="${m}" />
             <!--for a solid cylinder-->
-            <inertia ixx="${(m/12) * (3*r*r + l*l)}" ixy="0" ixz="0"
-                     iyy="${(m/12) * (3*r*r + l*l)}" iyz="0"
-                     izz="${(m/2) * (r*r)}" />
+            <inertia ixx="${(m/12.0) * (3*r*r + l*l)}" ixy="0" ixz="0"
+                     iyy="${(m/12.0) * (3*r*r + l*l)}" iyz="0"
+                     izz="${(m/2.0) * (r*r)}" />
         </inertial>
     </xacro:macro>

File: my_robot_description/urdf/mobile_base.xacro (robot description, xacro)
@@ -21,6 +21,7 @@
             <origin xyz="0 0 ${base_height / 2.0}" rpy="0 0 0" />
         </collision>
-        <xacro:box_inertia m="5.0" l="${base_length}" w="${base_width}" h="${base_height}"
+        <xacro:box_inertia m="5.0" l="${2*base_length}" w="${2*base_width}" h="${2*base_height}"
                            xyz="0 0 ${base_height / 2.0}" rpy="0 0 0" />
+        <!--multiplied inertial values we send by 2 because the robot was moving in place-->
     </link>
     <!--function. params not mandatory-->
@@ -40,5 +41,5 @@
                 <origin xyz="0 0 0" rpy="${pi / 2.0} 0 0" />
             </collision>
-            <xacro:cylinder_inertia m="1.0" r="${wheel_radius}" l="${wheel_length}"
+            <xacro:cylinder_inertia m="1.0" r="${2*wheel_radius}" l="${2*wheel_length}"
                                  xyz="0 0 0" rpy="${pi / 2.0} 0 0" />
         </link>
@@ -60,5 +61,5 @@
             <origin xyz="0 0 0" rpy="0 0 0" />
         </collision>
-        <xacro:sphere_inertia m="0.5" r="${wheel_radius / 2.0}"
+        <xacro:sphere_inertia m="0.5" r="${2*wheel_radius / 2.0}"
                               xyz="0 0 0" rpy="0 0 0" />
     </link>

File: my_robot_description/urdf/my_robot.urdf.xacro (robot description, xacro)
@@ -2,5 +2,7 @@
 <robot name="my_robot" xmlns:xacro="http://www.ros.org/wiki/xacro">
     <!--colcon build symlink install, again after creating files-->
+    <!--include order is important-->
     <xacro:include filename="common_properties.xacro" />
     <xacro:include filename="mobile_base.xacro" />
+    <xacro:include filename="mobile_base_gazebo.xacro" />
 </robot>
