Commit message: added collision properties

File: my_robot_description/install/my_robot_description/share/my_robot_description/urdf/mobile_base.xacro (robot description, xacro)
@@ -22,5 +22,5 @@
         </collision>
         <xacro:box_inertia m="5.0" l="${base_length}" w="${base_width}" h="${base_height}"
-                           xyz="0 0 ${base_height / 2.0}" rpy="0 0 0" />
+                           xyz="${base_height / 2.0}" rpy="0 0 0" />
     </link>
     <!--function. params not mandatory-->
@@ -34,10 +34,4 @@
                 <material name="gray" />
             </visual>
-            <collision>
-                <geometry>
-                    <cylinder radius="${wheel_radius}" length="${wheel_length}" />
-                </geometry>
-                <origin xyz="0 0 0" rpy="${pi / 2.0} 0 0" />
-            </collision>
             <xacro:cylinder_inertia m="1.0" r="${wheel_radius}" l="${wheel_length}"
                                  xyz="0 0 0" rpy="${pi / 2.0} 0 0" />
@@ -54,10 +48,4 @@
             <material name="gray" />
         </visual>
-        <collision>
-            <geometry>
-                <sphere radius="${wheel_radius / 2.0}" />
-            </geometry>
-            <origin xyz="0 0 0" rpy="0 0 0" />
-        </collision>
         <xacro:sphere_inertia m="0.5" r="${wheel_radius / 2.0}"
                               xyz="0 0 0" rpy="0 0 0" />
